Commit message: Working G1

File: robot_model/g1/g1_29dof_lock_waist.urdf (robot description, URDF)
Before this commit: robot g1_29dof_lock_waist, 43 links, 42 joints
Links:
- link left_ankle_roll_link: geometry collision box size=0.2 0.06 0.02; visual mesh filename=meshes/left_ankle_roll_link.STL
- link right_ankle_roll_link: geometry collision box size=0.2 0.06 0.02; visual mesh filename=meshes/right_ankle_roll_link.STL
Joints:
- joint waist_yaw_joint: limit lower=-2.618 upper=2.618 effort=88 velocity=32 -> lower=0 upper=0 effort=88 velocity=32

File: robot_model/g1/g1_simple_collisions.urdf (robot description, URDF)
Before this commit: robot g1, 47 links, 46 joints
Links:
- removed link left_elbow_pitch_link
- removed link left_elbow_roll_link
- removed link left_five_link
- removed link left_four_link
- removed link left_one_link
- removed link left_palm_link
- removed link left_six_link
- removed link left_three_link
- removed link left_two_link
- removed link left_zero_link
- removed link right_elbow_pitch_link
- removed link right_elbow_roll_link
- removed link right_five_link
- removed link right_four_link
- removed link right_one_link
- removed link right_palm_link
- removed link right_six_link
- removed link right_three_link
- removed link right_two_link
- removed link right_zero_link
- added link left_elbow_link, mass 0.6; collision mesh filename=meshes/left_elbow_link.STL; visual mesh filename=meshes/left_elbow_link.STL
- added link left_rubber_hand, mass 0.170; visual mesh filename=meshes/left_rubber_hand.STL
- added link left_wrist_pitch_link, mass 0.48404956; collision mesh filename=meshes/left_wrist_pitch_link.STL; visual mesh filename=meshes/left_wrist_pitch_link.STL
- added link left_wrist_roll_link, mass 0.08544498; collision mesh filename=meshes/left_wrist_roll_link.STL; visual mesh filename=meshes/left_wrist_roll_link.STL
- added link left_wrist_yaw_link, mass 0.08457647; collision mesh filename=meshes/left_wrist_yaw_link.STL; visual mesh filename=meshes/left_wrist_yaw_link.STL
- added link right_elbow_link, mass 0.6; collision mesh filename=meshes/right_elbow_link.STL; visual mesh filename=meshes/right_elbow_link.STL
- added link right_rubber_hand, mass 0.170; visual mesh filename=meshes/right_rubber_hand.STL
- added link right_wrist_pitch_link, mass 0.48404956; collision mesh filename=meshes/right_wrist_pitch_link.STL; visual mesh filename=meshes/right_wrist_pitch_link.STL
- added link right_wrist_roll_link, mass 0.08544498; collision mesh filename=meshes/right_wrist_roll_link.STL; visual mesh filename=meshes/right_wrist_roll_link.STL
- added link right_wrist_yaw_link, mass 0.08457647; collision mesh filename=meshes/right_wrist_yaw_link.STL; visual mesh filename=meshes/right_wrist_yaw_link.STL
Joints:
- removed joint left_elbow_pitch_joint
- removed joint left_elbow_roll_joint
- removed joint left_five_joint
- removed joint left_four_joint
- removed joint left_one_joint
- removed joint left_palm_joint
- removed joint left_six_joint
- removed joint left_three_joint
- removed joint left_two_joint
- removed joint left_zero_joint
- removed joint right_elbow_pitch_joint
- removed joint right_elbow_roll_joint
- removed joint right_five_joint
- removed joint right_four_joint
- removed joint right_one_joint
- removed joint right_palm_joint
- removed joint right_six_joint
- removed joint right_three_joint
- removed joint right_two_joint
- removed joint right_zero_joint
- added joint left_elbow_joint: type revolute, parent left_shoulder_yaw_link, child left_elbow_link, origin xyz=0.015783 0 -0.080518 rpy=0 0 0, axis 0 1 0, limit lower=-1.0472 upper=2.0944 effort=25 velocity=37
- added joint left_hand_palm_joint: type fixed, parent left_wrist_yaw_link, child left_rubber_hand, origin xyz=0.0415 0.003 0 rpy=0 0 0
- added joint left_wrist_pitch_joint: type revolute, parent left_wrist_roll_link, child left_wrist_pitch_link, origin xyz=0.038 0 0 rpy=0 0 0, axis 0 1 0, limit lower=-1.614429558 upper=1.614429558 effort=5 velocity=22
- added joint left_wrist_roll_joint: type revolute, parent left_elbow_link, child left_wrist_roll_link, origin xyz=0.100 0.00188791 -0.010 rpy=0 0 0, axis 1 0 0, limit lower=-1.972222054 upper=1.972222054 effort=25 velocity=37
- added joint left_wrist_yaw_joint: type revolute, parent left_wrist_pitch_link, child left_wrist_yaw_link, origin xyz=0.046 0 0 rpy=0 0 0, axis 0 0 1, limit lower=-1.614429558 upper=1.614429558 effort=5 velocity=22
- added joint right_elbow_joint: type revolute, parent right_shoulder_yaw_link, child right_elbow_link, origin xyz=0.015783 0 -0.080518 rpy=0 0 0, axis 0 1 0, limit lower=-1.0472 upper=2.0944 effort=25 velocity=37
- added joint right_hand_palm_joint: type fixed, parent right_wrist_yaw_link, child right_rubber_hand, origin xyz=0.0415 -0.003 0 rpy=0 0 0
- added joint right_wrist_pitch_joint: type revolute, parent right_wrist_roll_link, child right_wrist_pitch_link, origin xyz=0.038 0 0 rpy=0 0 0, axis 0 1 0, limit lower=-1.614429558 upper=1.614429558 effort=5 velocity=22
- added joint right_wrist_roll_joint: type revolute, parent right_elbow_link, child right_wrist_roll_link, origin xyz=0.100 -0.00188791 -0.010 rpy=0 0 0, axis 1 0 0, limit lower=-1.972222054 upper=1.972222054 effort=25 velocity=37
- added joint right_wrist_yaw_joint: type revolute, parent right_wrist_pitch_link, child right_wrist_yaw_link, origin xyz=0.046 0 0 rpy=0 0 0, axis 0 0 1, limit lower=-1.614429558 upper=1.614429558 effort=5 velocity=22
- joint torso_joint: limit lower=-2.618 upper=2.618 effort=88 velocity=32 -> lower=0 upper=0 effort=88 velocity=32

Commit message: Add cone viz and mujoco fix
* Add forces from croc to plot and viz in foxglove
* Manual merge of UI launcher
* Add mujoco switch gains on "P" keystroke
* Add dynamic CoM tracking

File: robot_model/g1/g1_29dof_lock_waist.urdf (robot description, URDF)
Before this commit: robot g1_29dof_lock_waist, 43 links, 42 joints
Links:
- added link torso_primitive_shape, mass 1e-9
Joints:
- added joint torso_primitive_shape_joint: type fixed, parent torso_link, child torso_primitive_shape, origin xyz=0.0039635 0.0 0.15 rpy=0 0 0
